File: BrainHat.kicad_pcb (KiCad board)
At the start: 2 copper layers, 48.2 x 49.8 mm, 31 parts, among them J1 Electrodes, J2 Output, J3 Power, J4 Status, U1 AD8232, U2 TS5A3159ADBVR

Commit message: YAAAA
Parts:
- added C10: 100nF, Capacitor_SMD:C_1210_3225Metric, F.Cu at (173.5, 81.0)
- added C11: 100nF, Capacitor_SMD:C_1210_3225Metric, F.Cu at (198.8, 89.3)
- added C12: 100nF, Capacitor_SMD:C_1210_3225Metric, F.Cu at (198.8, 94.8)
- added C9: 1nF, Capacitor_THT:C_Disc_D6.0mm_W4.4mm_P5.00mm, F.Cu at (153.5, 79.4)
- added D5: XL-1608UGC-04, LED_SMD:LED_0603_1608Metric, F.Cu at (145.2, 86.8)
- added H1: MountingHole, MountingHole:MountingHole_2.2mm_M2, F.Cu at (138.0, 59.0)
- added H2: MountingHole, MountingHole:MountingHole_2.2mm_M2, F.Cu at (137.0, 94.0)
- added H3: MountingHole, MountingHole:MountingHole_2.2mm_M2, F.Cu at (184.0, 60.0)
- added H4: MountingHole, MountingHole:MountingHole_2.2mm_M2, F.Cu at (198.6, 80.6)
- added R14: 10k, Resistor_SMD:R_1206_3216Metric, F.Cu at (194.4, 83.8)
- added R15: 10M±1%, Resistor_THT:R_Axial_DIN0309_L9.0mm_D3.2mm_P15.24mm_Horizontal, F.Cu at (153.0, 89.6)
- added R16: 330k, Resistor_SMD:R_0402_1005Metric, F.Cu at (178.2, 89.6)
- added R17: 330k, Resistor_SMD:R_0402_1005Metric, F.Cu at (178.2, 92.0)
- added R18: 10M±1%, Resistor_THT:R_Axial_DIN0309_L9.0mm_D3.2mm_P15.24mm_Horizontal, F.Cu at (153.0, 95.0)
- added R19: 10k, Resistor_SMD:R_1206_3216Metric, F.Cu at (189.6, 96.6)
- added U3: TS5A3159ADBVR, Package_TO_SOT_SMD:SOT-23-6, F.Cu at (174.2, 86.6)
- added U4: SN74LV1T34DBV, Package_TO_SOT_SMD:SOT-23-5, F.Cu at (194.0, 89.6)
- added U5: SN74LV1T34DBV, Package_TO_SOT_SMD:SOT-23-5, F.Cu at (194.0, 94.6)
- C1: value CA45-B6R3K107T -> 100nF; footprint Capacitor_Tantalum_SMD:CP_EIA-3528-21_Kemet-B -> Capacitor_SMD:C_1210_3225Metric
- C2: value ECHU1C104GX5 -> 10nF; footprint Capacitor_SMD:C_1210_3225Metric -> Capacitor_THT:C_Disc_D12.0mm_W4.4mm_P7.75mm
- C3: value CC0402JRX7R9BB102 -> 14pF
- C4, C8: value ECHU1C104GX5 -> 100nF
- C5: value 0402CG140J500NT -> 220uF; footprint Capacitor_SMD:C_0402_1005Metric -> Capacitor_SMD:C_Elec_6.3x5.4
- C6: value CA45-A010K106T -> 220uF; footprint Capacitor_Tantalum_SMD:CP_EIA-3216-12_Kemet-S -> Capacitor_SMD:C_Elec_6.3x5.4
- C7: value CA45-A010K106T -> 1uF; footprint Capacitor_Tantalum_SMD:CP_EIA-3216-12_Kemet-S -> Capacitor_THT:C_Disc_D5.1mm_W3.2mm_P5.00mm
- D3: value XL-1608UGC-04 -> XL-2012UWC; footprint LED_SMD:LED_0603_1608Metric -> LED_SMD:LED_0805_2012Metric
- J1: value Electrodes -> Power
- J2, J4: footprint Connector_PinSocket_2.54mm:PinSocket_1x03_P2.54mm_Vertical -> Connector_PinSocket_2.54mm:PinSocket_1x04_P2.54mm_Vertical
- J3: value Power -> Electrodes; footprint Connector_PinSocket_2.54mm:PinSocket_1x04_P2.54mm_Vertical -> Connector_PinHeader_2.54mm:PinHeader_1x06_P2.54mm_Vertical
- R1: value ARG03BTC1002 -> 10M±1%; footprint Resistor_SMD:R_0603_1608Metric -> Resistor_THT:R_Axial_DIN0309_L9.0mm_D3.2mm_P15.24mm_Horizontal
- R10: value 0603WAD3302T5E -> 10M±1%; footprint Resistor_SMD:R_0603_1608Metric -> Resistor_THT:R_Axial_DIN0309_L9.0mm_D3.2mm_P15.24mm_Horizontal
- R11: value CF1/6W-7.5KΩ±5%T52 -> 412k; footprint Personal:R_Axial_DIN0207_L6.3mm_D2.5mm_P5.08mm_Horizontal -> Resistor_SMD:R_2010_5025Metric
- R12, R13: value 1206W4F1002T5E -> 330k; footprint Resistor_SMD:R_1206_3216Metric -> Resistor_SMD:R_0402_1005Metric
- R2: value SCR0402J330K -> 10M±1%; footprint Resistor_SMD:R_0402_1005Metric -> Resistor_THT:R_Axial_DIN0309_L9.0mm_D3.2mm_P15.24mm_Horizontal
- R3: value 0603WAD3302T5E -> 604; footprint Resistor_SMD:R_0603_1608Metric -> Resistor_SMD:R_0402_1005Metric
- R4: value ARG03BTC1002 -> 10k; footprint Resistor_SMD:R_0603_1608Metric -> Resistor_SMD:R_1206_3216Metric
- R5: value SCR0402J330K -> 1.2M
- R6: value ARG05DTC1600 -> 1k; footprint Resistor_SMD:R_0805_2012Metric -> Resistor_SMD:R_0402_1005Metric
- R7: value 1206W4F1002T5E -> 1.58M; footprint Resistor_SMD:R_1206_3216Metric -> Resistor_SMD:R_0402_1005Metric
- R8: value 1206W4F1002T5E -> 1.2M; footprint Resistor_SMD:R_1206_3216Metric -> Resistor_SMD:R_0402_1005Metric
- R9: value ARG05DTC1600 -> 330; footprint Resistor_SMD:R_0805_2012Metric -> Resistor_SMD:R_0402_1005Metric
- U2: value TS5A3159ADBVR -> ADS1251; footprint Package_TO_SOT_SMD:SOT-23-6 -> Package_SO:MSOP-8_3x3mm_P0.65mm
- moved R9 64.8 mm to (201.2, 74.6), turned to -90 degrees
- moved C7 60.2 mm to (193.8, 69.0), turned to 0 degrees
- moved U2 49.7 mm to (196.0, 74.2), turned to 180 degrees
- moved C3 46.3 mm to (185.4, 65.4), turned to 0 degrees
- moved C4 42.3 mm to (196.4, 63.8), turned to 0 degrees
- moved C6 39.0 mm to (147.5, 68.8), turned to 0 degrees
- moved D4 36.8 mm to (141.0, 86.8), turned to 0 degrees
- moved D3 34.4 mm to (135.1, 87.4), turned to 0 degrees
- moved C8 32.9 mm to (148.0, 74.4)
- moved D2 32.2 mm to (141.0, 83.6)
- moved R12 31.4 mm to (178.0, 81.8), turned to 0 degrees
- moved R11 31.2 mm to (166.0, 79.8), turned to 0 degrees
- moved D1 30.8 mm to (135.1, 83.8)
- moved C5 30.4 mm to (137.0, 68.8), turned to 0 degrees
- moved R4 29.3 mm to (189.2, 64.2), turned to 180 degrees
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Connections:
- C1 pad 1: HPDRIVE1 -> +3.3V
- C1 pad 2: HPSENSE1 -> GND
- C3 pad 1: RLDFB1 -> Aref
- C3 pad 2: RLD1 -> UFOUT1
- C4 pad 1: +3.3V -> +5V
- C5 pad 1: Aref -> REFOUT1
- C5 pad 2: UFOUT1 -> Net-(C5-Pad2)
- C6 pad 1: Net-(C6-Pad1) -> Net-(C5-Pad2)
- C7 pad 1: REFOUT1 -> +5V
- C7 pad 2: Net-(C6-Pad1) -> GND
- C8 pad 1: +3.3V -> HPDRIVE1
- C8 pad 2: GND -> HPSENSE1
- D1 pad 2: connected1 -> connectedI
- D3 pad 1: switch -> GND
- D3 pad 2: +3.3V -> connectedR
- D4 pad 1: GND -> switch
- D4 pad 2: switch -> +3.3V
- J1 pad 1: Ge -> +5V
- J1 pad 2: 1e -> +3.3V
- J1 pad 3: Ze -> Aref
- J1 pad 4: 2e -> GND
- J2 pad 2: unconnected-(J2-Pin_2-Pad2) -> SCLK
- J2 pad 3: unconnected-(J2-Pin_3-Pad3) -> DOUT/~{DRDY}
- J3 pad 1: unconnected-(J3-Pin_1-Pad1) -> Net-(J3-Pin_1)
- J3 pad 2: +3.3V -> Net-(J3-Pin_2)
- J3 pad 3: Aref -> unconnected-(J3-Pin_3-Pad3)
- J3 pad 4: GND -> Net-(J3-Pin_4)
- J4 pad 1: connected1 -> connectedR
- J4 pad 2: shutdown -> connectedI
- J4 pad 3: switch -> 5Vshutdown
- R1 pad 1: +3.3V -> Vref
- R1 pad 2: Vref -> GND
- R10 pad 1: Net-(C6-Pad1) -> +3.3V
- R10 pad 2: OPAMP+1 -> 1e
- R11 pad 1: REFOUT1 -> RLD1
- R11 pad 2: OPAMP-1 -> Ge
- R12 pad 1: GND -> Ge
- R12 pad 2: switch -> Net-(J3-Pin_1)
- R13 pad 1: shutdown -> 1e
- R13 pad 2: +3.3V -> Net-(J3-Pin_2)
- R2 pad 1: IAOUT1 -> +3.3V
- R2 pad 2: HPSENSE1 -> Vref
- R3 pad 1: IAOUT1 -> UFOUT1
- R3 pad 2: Net-(C6-Pad1) -> OPAMP-1
- R4 pad 1: Vref -> 1o
- R4 pad 2: GND -> UFOUT1
- R5 pad 1: Ge -> IAOUT1
- R5 pad 2: RLD1 -> Net-(C5-Pad2)
- R6 pad 1: IAOUT1 -> OPAMP-1
- R6 pad 2: Net-(C6-Pad1) -> REFOUT1
- R7 pad 1: OPAMP-1 -> HPSENSE1
- R7 pad 2: 1o -> IAOUT1
- R8 pad 1: UFOUT1 -> Net-(C5-Pad2)
- R8 pad 2: 1o -> OPAMP+1
- R9 pad 1: Net-(C6-Pad1) -> UFOUT1
- R9 pad 2: OPAMP+1 -> Net-(U2-IN+)
- U1 pad 11: unconnected-(U1-LOD--Pad11) -> connectedR
- U1 pad 12: connected1 -> connectedI
- U1 pad 14: +3.3V -> GND
- U1 pad 15: GND -> +3.3V
- U1 pad 2: Ze -> Ie
- U1 pad 3: Ie -> Re
- U2 pad 1: 2e -> Net-(U2-IN+)
- U2 pad 2: GND -> +3.3V
- U2 pad 3: 1e -> +5V
- U2 pad 4: Ie -> CLK
- U2 pad 5: +3.3V -> DOUT/~{DRDY}
- U2 pad 6: switch -> SCLK
Routing:
- net connectedI: track 0.00 -> 118.2 mm
- net +3.3V: track 98.4 -> 214.3 mm
- net connectedR: track 0.00 -> 108.7 mm
- net connected1: track 107.0 -> 0.00 mm
- net Re: track 0.00 -> 74.7 mm, vias 0 -> 1
- net GND: track 14.2 -> 83.9 mm, vias 43 -> 62
- net UFOUT1: track 33.0 -> 85.8 mm
- net Net-(C6-Pad1): track 44.2 -> 0.00 mm, vias 2 -> 0
- net Ge: track 49.7 -> 10.0 mm
- net +5V: track 0.00 -> 28.5 mm, vias 0 -> 1
- net HPDRIVE1: track 3.88 -> 31.7 mm, vias 0 -> 2
- net OPAMP-1: track 11.1 -> 38.9 mm, vias 2 -> 0
- net HPSENSE1: track 7.87 -> 34.1 mm, vias 0 -> 2
- net Net-(C5-Pad2): track 0.00 -> 19.6 mm
- net shutdown: track 98.1 -> 79.1 mm, vias 2 -> 3
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Other:
- board size 48.2 x 49.8 mm -> 73 x 51.2 mm
- board text added: "->Ie"
- board text added: "1e"
- board text added: "2e"
- board text added: "Art by the amazing @abhay in the hackclub slack!"
- board text added: "Brain Hat R2"
- board text added: "Ie"
- board text added: "Re"
- board text removed: "1E"
- board text removed: "2E"
- board text removed: "3.3V"
- board text removed: "Aref"
- board text removed: "Brain Hat"
- board text removed: "Conn"
- board text removed: "Connected"
- board text removed: "Electrode 1"
- board text removed: "Electrode 2"
- board text removed: "Electrodes"
- board text removed: "GE"
- board text removed: "GND"
- board text removed: "Out"
- board text removed: "Selected:"
- board text removed: "Shtdn"
- board text removed: "Switch"
- board text removed: "ZE"
- board text removed: "hat by arif fajar yulianto from Noun Project (CC BY 3.0) Brain by ridhobadal from Noun Project (CC BY 3.0)"

Commit message: Silkscreen
Other:
- board text added: "+3.3V"
- board text added: "+5V"
- board text added: "Aref"
- board text added: "CLK"
- board text added: "DOUT ~{DRDY}"
- board text added: "GND"
- board text added: "Ge"
- board text added: "Ic"
- board text added: "Out"
- board text added: "Rc"
- board text added: "SCLK"
- board text added: "SW"
- board text added: "~{SD}"
Changed lines of the file:
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@@
 		(layer "Edge.Cuts")
+	)
+	(gr_text "SCLK"
+		(at 187.8 71.4 0)
+		(layer "F.SilkS")
+		(effects
+			(font
+				(size 1 1)
+				(thickness 0.2)
+				(bold yes)
+			)
+			(justify right)
+		)
 	)
 	(gr_text "->Ie"
@@
 		)
 	)
+	(gr_text "2e"
+		(at 183.6 89.4 0)
+		(layer "F.SilkS")
+		(effects
+			(font
+				(size 1 1)
+				(thickness 0.2)
+				(bold yes)
+			)
+			(justify left)
+		)
+	)
+	(gr_text "DOUT\n~{DRDY}"
+		(at 187.8 74.2 0)
+		(layer "F.SilkS")
+		(effects
+			(font
+				(size 0.8 1)
+				(thickness 0.2)
+				(bold yes)
+			)
+			(justify right)
+		)
+	)
+	(gr_text "GND"
+		(at 179.8 77.2 0)
+		(layer "F.SilkS")
+		(effects
+			(font
+				(size 1 1)
+				(thickness 0.2)
+				(bold yes)
+			)
+			(justify right bottom)
+		)
+	)
 	(gr_text "Ie"
 		(at 134.2 82.4 0)
@@
 		)
 	)
+	(gr_text "Out"
+		(at 187.6 68.8 0)
+		(layer "F.SilkS")
+		(effects
+			(font
+				(size 1 1)
+				(thickness 0.2)
+				(bold yes)
+			)
+			(justify right)
+		)
+	)
+	(gr_text "Aref"
+		(at 179.8 74.8 0)
+		(layer "F.SilkS")
+		(effects
+			(font
+				(size 1 1)
+				(thickness 0.2)
+				(bold yes)
+			)
+			(justify right bottom)
+		)
+	)
+	(gr_text "+5V"
+		(at 179.8 69.8 0)
+		(layer "F.SilkS")
+		(effects
+			(font
+				(size 1 1)
+				(thickness 0.2)
+				(bold yes)
+			)
+			(justify right bottom)
+		)
+	)
+	(gr_text "Ge"
+		(at 183.6 81.8 0)
+		(layer "F.SilkS")
+		(effects
+			(font
+				(size 1 1)
+				(thickness 0.2)
+				(bold yes)
+			)
+			(justify left)
+		)
+	)
+	(gr_text "+3.3V"
+		(at 179.8 72.2 0)
+		(layer "F.SilkS")
+		(effects
+			(font
+				(size 1 1)
+				(thickness 0.2)
+				(bold yes)
+			)
+			(justify right bottom)
+		)
+	)
+	(gr_text "CLK"
+		(at 187.8 76.8 0)
+		(layer "F.SilkS")
+		(effects
+			(font
+				(size 1 1)
+				(thickness 0.2)
+				(bold yes)
+			)
+			(justify right)
+		)
+	)
+	(gr_text "1e"
+		(at 183.6 84.4 0)
+		(layer "F.SilkS")
+		(effects
+			(font
+				(size 1 1)
+				(thickness 0.2)
+				(bold yes)
+			)
+			(justify left)
+		)
+	)
 	(gr_text "Art by the amazing @abhay in the hackclub slack!"
 		(at 138.7 101.1 0)
@@
 		)
 	)
+	(gr_text "Ic"
+		(at 188 86.8 0)
+		(layer "F.SilkS")
+		(effects
+			(font
+				(size 1 1)
+				(thickness 0.2)
+				(bold yes)
+			)
+			(justify right)
+		)
+	)
+	(gr_text "Rc"
+		(at 188 84.4 0)
+		(layer "F.SilkS")
+		(effects
+			(font
+				(size 1 1)
+				(thickness 0.2)
+				(bold yes)
+			)
+			(justify right)
+		)
+	)
 	(gr_text "On"
 		(at 140.2 82.5 0)
@@
 		)
 	)
+	(gr_text "~{SD}"
+		(at 188 89.6 0)
+		(layer "F.SilkS")
+		(effects
+			(font
+				(size 1 1)
+				(thickness 0.2)
+				(bold yes)
+			)
+			(justify right)
+		)
+	)
 	(gr_text "Brain Hat R2"
 		(at 192.4 59 0)
@@
 		)
 	)
+	(gr_text "SW"
+		(at 188 92 0)
+		(layer "F.SilkS")
+		(effects
+			(font
+				(size 1 1)
+				(thickness 0.2)
+				(bold yes)
+			)
+			(justify right)
+		)
+	)
+	(gr_text "Re"
+		(at 183.6 92 0)
+		(layer "F.SilkS")
+		(effects
+			(font
+				(size 1 1)
+				(thickness 0.2)
+				(bold yes)
+			)
+			(justify left)
+		)
+	)

Commit message: Changes
Parts:
- removed C7: 1uF, Capacitor_THT:C_Disc_D5.1mm_W3.2mm_P5.00mm
- removed R9: 330, Resistor_SMD:R_0402_1005Metric
- U2: value ADS1251 -> ADS1115IDGS; footprint Package_SO:MSOP-8_3x3mm_P0.65mm -> Package_SO:TSSOP-10_3x3mm_P0.5mm
- moved H4 16.7 mm to (208.0, 94.4)
- moved H3 9.77 mm to (193.0, 56.2)
Connections:
- C4 pad 1: +5V -> +3.3V
- J1 pad 1: +5V -> unconnected-(J1-Pin_1-Pad1)
- J2 pad 2: SCLK -> SCL
- J2 pad 3: DOUT/~{DRDY} -> ALERT
- J2 pad 4: CLK -> SDA
- U2 pad 1: Net-(U2-IN+) -> GND
- U2 pad 2: +3.3V -> ALERT
- U2 pad 3: +5V -> GND
- U2 pad 4: CLK -> UFOUT1
- U2 pad 5: DOUT/~{DRDY} -> unconnected-(U2-AIN1-Pad5)
- U2 pad 6: SCLK -> unconnected-(U2-AIN2-Pad6)
- U2 pad 7: GND -> unconnected-(U2-AIN3-Pad7)
Routing:
- net +5V: track 28.5 -> 0.00 mm, vias 1 -> 0
- net +3.3V: track 214.3 -> 230.0 mm
- net ALERT: track 0.00 -> 15.6 mm
- net CLK: track 9.74 -> 0.00 mm
- net SCL: track 0.00 -> 8.04 mm
- net SCLK: track 7.71 -> 0.00 mm
- net SDA: track 0.00 -> 7.07 mm
- net DOUT/~{DRDY}: track 4.47 -> 0.00 mm
- net GND: track 83.9 -> 80.3 mm, vias 62 -> 68
- net Net-(U2-IN+): track 3.02 -> 0.00 mm
- net shutdown: track 79.1 -> 80.5 mm
- net UFOUT1: track 85.8 -> 85.2 mm
Other:
- board size 73 x 51.2 mm -> 86 x 51.2 mm
- board text added: "ALERT"
- board text added: "SCL"
- board text added: "SDA"
- board text removed: "+5V"
- board text removed: "CLK"
- board text removed: "DOUT ~{DRDY}"
- board text removed: "SCLK"

Commit message: Redid PCB again
Parts:
- removed C11, C12, C8: 100nF, Capacitor_SMD:C_1210_3225Metric
- removed D3: XL-2012UWC, LED_SMD:LED_0805_2012Metric
- removed D5: XL-1608UGC-04, LED_SMD:LED_0603_1608Metric
- removed R17: 330k, Resistor_SMD:R_0402_1005Metric
- removed R18: 10M±1%, Resistor_THT:R_Axial_DIN0309_L9.0mm_D3.2mm_P15.24mm_Horizontal
- removed R19: 10k, Resistor_SMD:R_1206_3216Metric
- removed U3: TS5A3159ADBVR, Package_TO_SOT_SMD:SOT-23-6
- removed U5: SN74LV1T34DBV, Package_TO_SOT_SMD:SOT-23-5
- added C7: 220uF, Capacitor_SMD:C_Elec_6.3x5.4, F.Cu at (186.1, 72.9)
- added TP1: TestPoint, TestPoint:TestPoint_Pad_D1.5mm, F.Cu at (181.6, 80.3)
- added TP10: TestPoint, TestPoint:TestPoint_Pad_D1.5mm, F.Cu at (154.1, 100.1)
- added TP12: TestPoint, TestPoint:TestPoint_Pad_D1.5mm, F.Cu at (166.8, 90.8)
- added TP13: TestPoint, TestPoint:TestPoint_Pad_D1.5mm, F.Cu at (197.5, 80.5)
- added TP16: TestPoint, TestPoint:TestPoint_Pad_D1.5mm, F.Cu at (168.6, 74.7)
- added TP2: TestPoint, TestPoint:TestPoint_Pad_D1.5mm, F.Cu at (177.8, 97.7)
- added TP3: TestPoint, TestPoint:TestPoint_Pad_D1.5mm, F.Cu at (175.9, 94.0)
- added TP4: TestPoint, TestPoint:TestPoint_Pad_D1.5mm, F.Cu at (184.7, 99.6)
- added TP5: TestPoint, TestPoint:TestPoint_Pad_D1.5mm, F.Cu at (184.6, 96.8)
- added TP6: TestPoint, TestPoint:TestPoint_Pad_D1.5mm, F.Cu at (161.6, 89.8)
- added TP7: TestPoint, TestPoint:TestPoint_Pad_D1.5mm, F.Cu at (161.6, 82.7)
- added TP8: TestPoint, TestPoint:TestPoint_Pad_D1.5mm, F.Cu at (161.9, 93.3)
- added TP9: TestPoint, TestPoint:TestPoint_Pad_D1.5mm, F.Cu at (181.6, 97.7)
- C10: value 100nF -> 14pF; footprint Capacitor_SMD:C_1210_3225Metric -> Capacitor_SMD:C_0402_1005Metric
- C2: value 10nF -> 100nF; footprint Capacitor_THT:C_Disc_D12.0mm_W4.4mm_P7.75mm -> Capacitor_SMD:C_1210_3225Metric
- C3: value 14pF -> 10nF; footprint Capacitor_SMD:C_0402_1005Metric -> Capacitor_SMD:C_0805_2012Metric
- C4: footprint Capacitor_SMD:C_1210_3225Metric -> Capacitor_THT:C_Disc_D7.5mm_W5.0mm_P5.00mm
- C6: value 220uF -> 1nF; footprint Capacitor_SMD:C_Elec_6.3x5.4 -> Capacitor_THT:C_Disc_D6.0mm_W4.4mm_P5.00mm
- C9: value 1nF -> 100nF; footprint Capacitor_THT:C_Disc_D6.0mm_W4.4mm_P5.00mm -> Capacitor_SMD:C_1210_3225Metric
- D1: value XL-2012UWC -> XL-1608UBC-04; footprint LED_SMD:LED_0805_2012Metric -> LED_SMD:LED_0603_1608Metric
- D2: value XL-1608UBC-04 -> XL-2012UWC; footprint LED_SMD:LED_0603_1608Metric -> LED_SMD:LED_0805_2012Metric
- D4: value XL-1608UGC-04 -> XL-2012UWC; footprint LED_SMD:LED_0603_1608Metric -> LED_SMD:LED_0805_2012Metric
- J2: value Output -> Status
- J4: value Status -> Output
- R1, R15: footprint Resistor_THT:R_Axial_DIN0309_L9.0mm_D3.2mm_P15.24mm_Horizontal -> Resistor_SMD:R_0402_1005Metric
- R10: value 10M±1% -> 412k; footprint Resistor_THT:R_Axial_DIN0309_L9.0mm_D3.2mm_P15.24mm_Horizontal -> Resistor_SMD:R_0402_1005Metric
- R11: value 412k -> 1.2M; footprint Resistor_SMD:R_2010_5025Metric -> Resistor_SMD:R_0402_1005Metric
- R12: value 330k -> 1.2M
- R13: value 330k -> 1k
- R14: value 10k -> 10M±1%; footprint Resistor_SMD:R_1206_3216Metric -> Resistor_SMD:R_0402_1005Metric
- R16: value 330k -> 10k; footprint Resistor_SMD:R_0402_1005Metric -> Resistor_SMD:R_1206_3216Metric
- R2: value 10M±1% -> 1.58M; footprint Resistor_THT:R_Axial_DIN0309_L9.0mm_D3.2mm_P15.24mm_Horizontal -> Resistor_SMD:R_0402_1005Metric
- R3: value 604 -> 10M±1%
- R4: value 10k -> 330k; footprint Resistor_SMD:R_1206_3216Metric -> Resistor_SMD:R_0402_1005Metric
- R5: value 1.2M -> 330k
- R6: value 1k -> 330k
- R7: value 1.58M -> 10k; footprint Resistor_SMD:R_0402_1005Metric -> Resistor_SMD:R_1206_3216Metric
- R8: value 1.2M -> 604
- U1: value AD8232 -> ADS1115IDGS; footprint Package_CSP:LFCSP-20-1EP_4x4mm_P0.5mm_EP2.5x2.5mm -> Package_SO:TSSOP-10_3x3mm_P0.5mm
- U2: value ADS1115IDGS -> AD8232; footprint Package_SO:TSSOP-10_3x3mm_P0.5mm -> Package_CSP:LFCSP-20-1EP_4x4mm_P0.5mm_EP2.5x2.5mm
- moved H1 59.1 mm to (196.0, 70.5)
- moved R6 56.0 mm to (190.7, 87.0), turned to 0 degrees
- moved H3 52.8 mm to (163.4, 99.9)
- moved C6 50.7 mm to (197.8, 75.6), turned to 180 degrees
- moved R5 50.1 mm to (190.7, 85.9)
- moved R2 48.6 mm to (187.7, 90.2), turned to 180 degrees
- moved D1 42.7 mm to (174.7, 99.7)
- moved C5 39.2 mm to (176.0, 72.9), turned to 180 degrees
- moved C2 38.9 mm to (157.8, 100.1), turned to 180 degrees
- moved R3 38.7 mm to (184.1, 90.1)
- moved R8 38.2 mm to (183.2, 83.0)
- moved R15 38.1 mm to (190.5, 83.1), turned to -90 degrees
- moved R10 38.0 mm to (190.7, 79.2)
- moved R1 37.7 mm to (182.1, 90.1)
- moved C4 34.4 mm to (188.6, 97.3), turned to 90 degrees
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Connections:
- C10 pad 1: +3.3V -> Aref
- C10 pad 2: GND -> UFOUT1
- C2 pad 1: Vref -> +3.3V
- C3 pad 1: Aref -> Vref
- C3 pad 2: UFOUT1 -> GND
- C4 pad 1: +3.3V -> HPDRIVE1
- C4 pad 2: GND -> HPSENSE1
- C5 pad 1: REFOUT1 -> Net-(C5-Pad1)
- C5 pad 2: Net-(C5-Pad2) -> UFOUT1
- C6 pad 1: Net-(C5-Pad2) -> RLDFB1
- C6 pad 2: UFOUT1 -> RLD1
- C9 pad 1: RLDFB1 -> +3.3V
- C9 pad 2: RLD1 -> GND
- D1 pad 1: GND -> shutdown
- D1 pad 2: connectedI -> +3.3V
- D2 pad 1: shutdown -> GND
- D2 pad 2: +3.3V -> connectedI
- D4 pad 1: switch -> GND
- D4 pad 2: +3.3V -> connectedR
- J2 pad 1: 1o -> connectedR
- J2 pad 2: SCL -> connectedI
- J2 pad 3: ALERT -> 5Vshutdown
- J2 pad 4: SDA -> unconnected-(J2-Pin_4-Pad4)
- J3 pad 2: Net-(J3-Pin_2) -> /E-
- J3 pad 3: unconnected-(J3-Pin_3-Pad3) -> /E+
- J3 pad 4: Net-(J3-Pin_4) -> unconnected-(J3-Pin_4-Pad4)
- J3 pad 5: Net-(J3-Pin_5) -> unconnected-(J3-Pin_5-Pad5)
- J4 pad 1: connectedR -> 1o
- J4 pad 2: connectedI -> SCL
- J4 pad 3: 5Vshutdown -> ALERT
- J4 pad 4: 5Vswitch -> SDA
- R1 pad 1: Vref -> +3.3V
- R1 pad 2: GND -> Vref
- R10 pad 1: +3.3V -> RLD1
- R10 pad 2: 1e -> Ge
- R11 pad 1: RLD1 -> IAOUT1
- R11 pad 2: Ge -> Net-(C5-Pad1)
- R12 pad 1: Ge -> Net-(C5-Pad1)
- R12 pad 2: Net-(J3-Pin_1) -> OPAMP+1
- R13 pad 1: 1e -> OPAMP-1
- R13 pad 2: Net-(J3-Pin_2) -> REFOUT1
- R14 pad 1: 5Vshutdown -> +3.3V
- R14 pad 2: +3.3V -> IN+
- R15 pad 2: 2e -> IN-
- R16 pad 1: 2e -> 1o
- R16 pad 2: Net-(J3-Pin_4) -> UFOUT1
- R2 pad 1: +3.3V -> HPSENSE1
- R2 pad 2: Vref -> IAOUT1
- R3 pad 1: UFOUT1 -> Vref
- R3 pad 2: OPAMP-1 -> GND
- R4 pad 1: 1o -> Ge
- R4 pad 2: UFOUT1 -> Net-(J3-Pin_1)
- R5 pad 1: IAOUT1 -> IN-
- R5 pad 2: Net-(C5-Pad2) -> /E-
- R6 pad 1: OPAMP-1 -> IN+
- R6 pad 2: REFOUT1 -> /E+
- R7 pad 1: HPSENSE1 -> 5Vshutdown
- R7 pad 2: IAOUT1 -> +3.3V
- R8 pad 1: Net-(C5-Pad2) -> UFOUT1
- R8 pad 2: OPAMP+1 -> OPAMP-1
- U1 pad 1: HPDRIVE1 -> GND
- U1 pad 10: UFOUT1 -> SCL
- U1 pad 2: Ie -> ALERT
- U1 pad 3: Re -> GND
- U1 pad 4: RLDFB1 -> UFOUT1
- U1 pad 5: RLD1 -> unconnected-(U1-AIN1-Pad5)
- U1 pad 6: IAOUT1 -> unconnected-(U1-AIN2-Pad6)
- U1 pad 7: OPAMP+1 -> unconnected-(U1-AIN3-Pad7)
- U1 pad 8: REFOUT1 -> +3.3V
- U1 pad 9: OPAMP-1 -> SDA
- U2 pad 1: GND -> HPDRIVE1
- U2 pad 10: SCL -> UFOUT1
- U2 pad 2: ALERT -> IN+
- U2 pad 3: GND -> IN-
- U2 pad 4: UFOUT1 -> RLDFB1
- U2 pad 5: unconnected-(U2-AIN1-Pad5) -> RLD1
- U2 pad 6: unconnected-(U2-AIN2-Pad6) -> IAOUT1
- U2 pad 7: unconnected-(U2-AIN3-Pad7) -> OPAMP+1
- U2 pad 8: +3.3V -> REFOUT1
- U2 pad 9: SDA -> OPAMP-1
Routing:
- net +3.3V: track 230.0 -> 103.0 mm, vias 3 -> 0
- net connectedI: track 118.2 -> 28.4 mm, vias 0 -> 1
- net connectedR: track 108.7 -> 20.7 mm, vias 0 -> 1
- net Re: track 74.7 -> 0.00 mm, vias 1 -> 0
- net switch: track 67.1 -> 0.00 mm, vias 4 -> 0
- net shutdown: track 80.5 -> 25.5 mm, vias 3 -> 4
- net GND: track 80.3 -> 43.3 mm, vias 68 -> 9
- net HPSENSE1: track 34.1 -> 4.06 mm, vias 2 -> 0
- net Ie: track 27.8 -> 0.00 mm, vias 2 -> 0
- net OPAMP-1: track 38.9 -> 11.7 mm, vias 0 -> 2
- net UFOUT1: track 85.2 -> 62.0 mm
- net REFOUT1: track 41.6 -> 18.5 mm, vias 0 -> 2
- net Aref: track 10.0 -> 31.3 mm
- net HPDRIVE1: track 31.7 -> 11.3 mm, vias 2 -> 0
- net Net-(C5-Pad2): track 19.6 -> 0.00 mm
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Other:
- board size 86 x 51.2 mm -> 50.6 x 40.3 mm
- board text added: "3.3V"
- board text added: "ADC: SCL"
- board text added: "Connected:"
- board text added: "Iconn"
- board text added: "Output"
- board text added: "Rconn"
- board text added: "Shdn"
- board text removed: "+3.3V"
- board text removed: "->Ie"
- board text removed: "1e"
- board text removed: "2e"
- board text removed: "Ge"
- board text removed: "Ic"
- board text removed: "On"
- board text removed: "Out"
- board text removed: "Rc"
- board text removed: "SCL"
- board text removed: "SW"
- board text removed: "~{SD}"

Commit message: Made a variety of changes
Parts:
- removed the TP12 at (166.8, 90.8)
- renumbered C5 to C1, C7 to C2, C10 to C3, C6 to C4, C1 to C5, C3 to C6, C4 to C7, C2 to C8, D2 to D1, D4 to D2, D1 to D3, H2 to H1, H1 to H2, J4 to J1, J1 to J3, J3 to J4, R16 to R1, R1 to R10, R14 to R11, R2 to R12, R5 to R13, R6 to R14, R7 to R15, R12 to R2, R11 to R3, R13 to R4, R10 to R5, R8 to R6, R4 to R7, R15 to R8, R3 to R9, TP16 to TP1, TP9 to TP10, TP10 to TP11, TP4 to TP12, TP7 to TP2, TP1 to TP3, TP13 to TP4, TP6 to TP5, TP8 to TP6, TP2 to TP7, TP3 to TP8, TP5 to TP9, U2 to U1, U1 to U2, U4 to U3
Routing:
- net IAOUT1: track 37.4 -> 38.1 mm
- net +3.3V: track 103.0 -> 103.7 mm
- net connectedI: track 28.4 -> 27.7 mm
Other:
- board text added: "3.3v"
- board text added: "Ge"
- board text added: "IAOUT"
- board text added: "SCL"
- board text added: "UFOut"
- board text added: "Vref"
